File: display.kicad_sch (KiCad schematic)
At the start: 17 parts, among them Q7 Q_NMOS_DGS, U12 E2266CS0C2

Commit message: schematic creation
Parts:
- D2, D3, D4: footprint (none) -> airsoft_controller:D-US2H-2
- L6: footprint (none) -> Inductor_SMD:L_1210_3225Metric_Pad1.42x2.65mm_HandSolder
- Q5: renamed from Q7; footprint (none) -> Package_TO_SOT_SMD:SOT-23; symbol Device:Q_NMOS_DGS -> Device:Q_NMOS_GSD
- R31: renamed from R33; footprint Resistor_SMD:R_0603_1608Metric -> Resistor_SMD:R_0603_1608Metric_Pad0.98x0.95mm_HandSolder
- renumbered C76 to C78, C77 to C79, C78 to C80, C79 to C81, C80 to C82, C81 to C83, C82 to C84, C83 to C85, C84 to C86, C85 to C87
Connections:
- net DP_RESE: now also Q5.2 (S); no longer Q5.3 (S)
- net GND: now also U12.25 (SHIELD), U12.26 (SHIELD)
- net at C87.2, D3.2 (A), L6.1: now also Q5.3 (D); no longer Q5.1 (D)
- net at U12.2 (GDR): now also Q5.1 (G); no longer Q5.2 (G)
Changed lines of the file:
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@@
   (junction (at 167.64 111.76) (diameter 0) (color 0 0 0 0)
   )
+  (junction (at 144.78 110.49) (diameter 0) (color 0 0 0 0)
+  )
   (junction (at 182.88 111.76) (diameter 0) (color 0 0 0 0)
   )
@@
     (stroke (width 0) (type default) (color 0 0 0 0))
   )
+  (wire (pts (xy 143.51 110.49) (xy 144.78 110.49))
+    (stroke (width 0) (type default) (color 0 0 0 0))
+  )
   (wire (pts (xy 182.88 93.98) (xy 182.88 104.14))
     (stroke (width 0) (type default) (color 0 0 0 0))
@@
   )
   (wire (pts (xy 160.02 99.06) (xy 172.72 99.06))
+    (stroke (width 0) (type default) (color 0 0 0 0))
+  )
+  (wire (pts (xy 144.78 110.49) (xy 147.32 110.49))
     (stroke (width 0) (type default) (color 0 0 0 0))
   )
@@
   (symbol (lib_id "Device:C") (at 182.88 107.95 180) (unit 1)
     (in_bom yes) (on_board yes)
-    (property "Reference" "C82" (id 0) (at 181.61 114.3 0)
+    (property "Reference" "C84" (id 0) (at 181.61 114.3 0)
       (effects (font (size 1.27 1.27)) (justify right))
     )
@@
     (pin "2")
   )
-  (symbol (lib_id "Device:Q_NMOS_DGS") (at 189.23 78.74 270) (mirror x) (unit 1)
-    (in_bom yes) (on_board yes)
-    (property "Reference" "Q7" (id 0) (at 189.23 71.12 90))
+  (symbol (lib_id "Device:Q_NMOS_GSD") (at 189.23 78.74 270) (mirror x) (unit 1)
+    (in_bom yes) (on_board yes)
+    (property "Reference" "Q5" (id 0) (at 189.23 71.12 90))
     (property "Value" "Q_NMOS_DGS" (id 1) (at 189.23 68.58 90))
-    (property "Footprint" "" (id 2) (at 191.77 73.66 0)
+    (property "Footprint" "Package_TO_SOT_SMD:SOT-23" (id 2) (at 191.77 73.66 0)
       (effects (font (size 1.27 1.27)) hide)
     )
@@
   (symbol (lib_id "power:GND") (at 196.85 96.52 0) (unit 1)
     (in_bom yes) (on_board yes) (fields_autoplaced)
-    (property "Reference" "#PWR093" (id 0) (at 196.85 102.87 0)
+    (property "Reference" "#PWR099" (id 0) (at 196.85 102.87 0)
       (effects (font (size 1.27 1.27)) hide)
     )
@@
   (symbol (lib_id "power:GND") (at 135.89 71.12 0) (unit 1)
     (in_bom yes) (on_board yes) (fields_autoplaced)
-    (property "Reference" "#PWR089" (id 0) (at 135.89 77.47 0)
+    (property "Reference" "#PWR095" (id 0) (at 135.89 77.47 0)
       (effects (font (size 1.27 1.27)) hide)
     )
@@
       (effects (font (size 1.27 1.27)) (justify right))
     )
-    (property "Footprint" "" (id 2) (at 196.85 85.09 0)
+    (property "Footprint" "airsoft_controller:D-US2H-2" (id 2) (at 196.85 85.09 0)
       (effects (font (size 1.27 1.27)) hide)
     )
@@
   (symbol (lib_id "power:GND") (at 144.78 110.49 0) (unit 1)
     (in_bom yes) (on_board yes) (fields_autoplaced)
-    (property "Reference" "#PWR091" (id 0) (at 144.78 116.84 0)
+    (property "Reference" "#PWR097" (id 0) (at 144.78 116.84 0)
       (effects (font (size 1.27 1.27)) hide)
     )
@@
   (symbol (lib_id "Device:C") (at 187.96 107.95 180) (unit 1)
     (in_bom yes) (on_board yes)
-    (property "Reference" "C83" (id 0) (at 186.69 114.3 0)
+    (property "Reference" "C85" (id 0) (at 186.69 114.3 0)
       (effects (font (size 1.27 1.27)) (justify right))
     )
@@
   (symbol (lib_id "power:+3.3V") (at 143.51 60.96 0) (unit 1)
     (in_bom yes) (on_board yes) (fields_autoplaced)
-    (property "Reference" "#PWR090" (id 0) (at 143.51 64.77 0)
+    (property "Reference" "#PWR096" (id 0) (at 143.51 64.77 0)
       (effects (font (size 1.27 1.27)) hide)
     )
@@
   (symbol (lib_id "Device:C") (at 162.56 107.95 180) (unit 1)
     (in_bom yes) (on_board yes)
-    (property "Reference" "C78" (id 0) (at 161.29 114.3 0)
+    (property "Reference" "C80" (id 0) (at 161.29 114.3 0)
       (effects (font (size 1.27 1.27)) (justify right))
     )
@@
   (symbol (lib_id "Device:C") (at 167.64 107.95 180) (unit 1)
     (in_bom yes) (on_board yes)
-    (property "Reference" "C79" (id 0) (at 166.37 114.3 0)
+    (property "Reference" "C81" (id 0) (at 166.37 114.3 0)
       (effects (font (size 1.27 1.27)) (justify right))
     )
@@
   (symbol (lib_id "Device:C") (at 139.7 71.12 270) (unit 1)
     (in_bom yes) (on_board yes)
-    (property "Reference" "C77" (id 0) (at 148.59 69.85 90)
+    (property "Reference" "C79" (id 0) (at 148.59 69.85 90)
       (effects (font (size 1.27 1.27)) (justify right))
     )
@@
   (symbol (lib_id "power:+3.3V") (at 213.36 81.28 0) (unit 1)
     (in_bom yes) (on_board yes) (fields_autoplaced)
-    (property "Reference" "#PWR095" (id 0) (at 213.36 85.09 0)
+    (property "Reference" "#PWR0101" (id 0) (at 213.36 85.09 0)
       (effects (font (size 1.27 1.27)) hide)
     )
@@
   (symbol (lib_id "power:GND") (at 172.72 77.47 0) (unit 1)
     (in_bom yes) (on_board yes) (fields_autoplaced)
-    (property "Reference" "#PWR092" (id 0) (at 172.72 83.82 0)
+    (property "Reference" "#PWR098" (id 0) (at 172.72 83.82 0)
       (effects (font (size 1.27 1.27)) hide)
     )
@@
       (effects (font (size 1.27 1.27)) (justify right))
     )
-    (property "Footprint" "" (id 2) (at 207.01 107.95 0)
+    (property "Footprint" "airsoft_controller:D-US2H-2" (id 2) (at 207.01 107.95 0)
       (effects (font (size 1.27 1.27)) hide)
     )
@@
   (symbol (lib_id "Device:C") (at 139.7 66.04 270) (unit 1)
     (in_bom yes) (on_board yes)
-    (property "Reference" "C76" (id 0) (at 148.59 64.77 90)
+    (property "Reference" "C78" (id 0) (at 148.59 64.77 90)
       (effects (font (size 1.27 1.27)) (justify right))
     )
@@
   (symbol (lib_id "Device:R") (at 177.8 76.2 90) (unit 1)
     (in_bom yes) (on_board yes)
-    (property "Reference" "R33" (id 0) (at 177.8 78.74 90))
+    (property "Reference" "R31" (id 0) (at 177.8 78.74 90))
     (property "Value" "0.47R" (id 1) (at 177.8 81.28 90))
-    (property "Footprint" "Resistor_SMD:R_0603_1608Metric" (id 2) (at 177.8 77.978 90)
+    (property "Footprint" "Resistor_SMD:R_0603_1608Metric_Pad0.98x0.95mm_HandSolder" (id 2) (at 177.8 77.978 90)
       (effects (font (size 1.27 1.27)) hide)
     )
@@
   (symbol (lib_id "Device:C") (at 177.8 107.95 180) (unit 1)
     (in_bom yes) (on_board yes)
-    (property "Reference" "C81" (id 0) (at 176.53 114.3 0)
+    (property "Reference" "C83" (id 0) (at 176.53 114.3 0)
       (effects (font (size 1.27 1.27)) (justify right))
     )
@@
       (effects (font (size 1.27 1.27)) (justify right))
     )
-    (property "Footprint" "" (id 2) (at 194.31 104.14 0)
+    (property "Footprint" "airsoft_controller:D-US2H-2" (id 2) (at 194.31 104.14 0)
       (effects (font (size 1.27 1.27)) hide)
     )
@@
   (symbol (lib_id "Device:C") (at 172.72 107.95 180) (unit 1)
     (in_bom yes) (on_board yes)
-    (property "Reference" "C80" (id 0) (at 171.45 114.3 0)
+    (property "Reference" "C82" (id 0) (at 171.45 114.3 0)
       (effects (font (size 1.27 1.27)) (justify right))
     )
@@
     (property "Reference" "L6" (id 0) (at 207.01 74.93 90))
     (property "Value" "10uH" (id 1) (at 207.01 77.47 90))
-    (property "Footprint" "" (id 2) (at 207.01 81.28 0)
+    (property "Footprint" "Inductor_SMD:L_1210_3225Metric_Pad1.42x2.65mm_HandSolder" (id 2) (at 207.01 81.28 0)
       (effects (font (size 1.27 1.27)) hide)
     )
@@
   (symbol (lib_id "power:GND") (at 198.12 113.03 0) (unit 1)
     (in_bom yes) (on_board yes) (fields_autoplaced)
-    (property "Reference" "#PWR094" (id 0) (at 198.12 119.38 0)
+    (property "Reference" "#PWR0100" (id 0) (at 198.12 119.38 0)
       (effects (font (size 1.27 1.27)) hide)
     )
@@
   (symbol (lib_id "Device:C") (at 196.85 92.71 180) (unit 1)
     (in_bom yes) (on_board yes)
-    (property "Reference" "C84" (id 0) (at 190.5 91.44 0)
+    (property "Reference" "C86" (id 0) (at 190.5 91.44 0)
       (effects (font (size 1.27 1.27)) (justify right))
     )
@@
   (symbol (lib_id "Device:C") (at 201.93 92.71 180) (unit 1)
     (in_bom yes) (on_board yes)
-    (property "Reference" "C85" (id 0) (at 205.74 91.44 0)
+    (property "Reference" "C87" (id 0) (at 205.74 91.44 0)
       (effects (font (size 1.27 1.27)) (justify right))
     )
@@
   (symbol (lib_id "airsoft_controller:E2266CS0C2") (at 144.78 92.71 0) (unit 1)
     (in_bom yes) (on_board yes)
-    (property "Reference" "U12" (id 0) (at 147.32 110.49 0)
+    (property "Reference" "U12" (id 0) (at 148.59 110.49 0)
       (effects (font (size 1.27 1.27)) (justify left))
     )
-    (property "Value" "E2266CS0C2" (id 1) (at 147.32 113.03 0)
+    (property "Value" "E2266CS0C2" (id 1) (at 148.59 113.03 0)
       (effects (font (size 1.27 1.27)) (justify left))
     )
@@
     (pin "23")
     (pin "24")
+    (pin "25")
+    (pin "26")
     (pin "3")
     (pin "4")
