File: airsoft_controller.kicad_pcb (KiCad board)
At the start: 2 copper layers, 180 x 100 mm, 333 parts, among them J1 Conn_01x07, J10 Conn_01x01, J11 USB_C_Receptacle, J12 Conn_01x03, J13 Conn_01x03, J14 Conn_01x05, J15 Conn_01x01, J2 Conn_01x03, J3 Conn_01x03, J4 Conn_01x01, J5 Conn_01x03, J6 Micro_SD_Card, J7 Conn_01x03, J8 Conn_01x02, J9 USB_C_Receptacle, Q1 Q_Dual_NMOS, Q10 Q_Dual_PMOS, Q11 Q_NMOS_DGS, Q12 Q_NMOS_DGS, Q13 Q_NMOS_DGS, Q14 Q_NMOS_DGS, Q15 Q_NMOS_DGS, Q16 Q_NMOS_DGS, Q2 Q_Dual_NMOS, Q3 Q_NMOS_DGS, Q4 Q_PMOS_DGS, Q5 Q_NMOS_DGS, Q6 Q_NMOS_DGS, Q7 Q_NMOS_DGS, Q8 Q_NMOS_DGS, Q9 Q_Dual_PMOS, SW1 MEMBRANE, SW2 MEMBRANE, SW3 MECH_SW, SW4 MEMBRANE, SW5 MEMBRANE, SW6 MEMBRANE, SW7 MEMBRANE, U1 CP2102N-Axx-xQFN20, U10 L96-M33, U11 RA-01SH, U12 E2266CS0C2, U13 TPD6S300A, U14 TPS65988, U15 TPD6S300A, U16 BQ29209DRBR, U17 LM358, U18 MP2229GQ-P, U19 MP2229GQ-P, U2 ESP32-S3-WROOM-1, U3 74HC595, U4 SN74HCS165, U5 TPS5403DR, U6 MP28167GQ-P, U7 BQ25731, U8 MC3479, U9 ST25DV04KC

Commit message: edited usb pcb part
Parts:
- added C153: 22uF, Capacitor_SMD:CP_Elec_5x5.3, F.Cu at (187.7, 77.2)
- added C162: 4.7uF, Capacitor_SMD:C_0603_1608Metric_Pad1.08x0.95mm_HandSolder, B.Cu at (204.7, 74.5)
- C88, C97: footprint Capacitor_SMD:C_1206_3216Metric_Pad1.33x1.80mm_HandSolder -> Capacitor_SMD:C_0805_2012Metric_Pad1.18x1.45mm_HandSolder; moved to B.Cu
- C89, D14, R34, R35, R36, R37, R38, R45, R46, R47, R48, R49, R50, R53, R54, R55, R56: moved to B.Cu
- D8: moved to F.Cu
- moved C145 247.6 mm to (191.7, 88.8)
- moved R73 244.9 mm to (192.5, 80.7)
- moved R77 244.8 mm to (189.3, 84.8)
- moved C141 243.3 mm to (195.8, 90.2)
- moved C143 239.0 mm to (193.1, 82.1)
- moved R66 238.9 mm to (189.3, 80.2)
- moved C149 234.3 mm to (191.9, 87.0)
- moved R45 233.7 mm to (203.4, 60.8), turned to 90 degrees
- moved R78 233.0 mm to (192.6, 84.8)
- moved C159 229.7 mm to (181.1, 85.9)
- moved R69 227.5 mm to (189.3, 81.8), turned to 180 degrees
- moved R50 227.4 mm to (205.3, 57.8), turned to -90 degrees
- moved R49 226.3 mm to (205.8, 60.2)
- moved R48 224.8 mm to (216.7, 56.2), turned to 180 degrees
- moved R53 222.6 mm to (205.8, 61.7), turned to 180 degrees
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Connections:
- J2 pad 1: /USB-C power controller/GPIO0 -> /USB-C power controller/GPIO3/HPD1
- J2 pad 3: /USB-C power controller/GPIO3/HPD1 -> /USB-C power controller/GPIO0
- R15 pad 1: +3V3 -> +3.3V
Routing:
- net /USB-C power controller/TPS_LDO_3V3: track 0.00 -> 24.3 mm, vias 0 -> 1
- net /USB-C power controller/USB1_VBUS: track 0.00 -> 22.9 mm, vias 0 -> 27
- net /USB-C power controller/TPS_SPI_POCI: track 0.00 -> 22.1 mm, vias 0 -> 1
- net Net-(Q12-Pad1): track 0.00 -> 21.0 mm, vias 0 -> 1
- net /USB-C power controller/USB1_SOURCE: track 0.00 -> 19.2 mm, vias 0 -> 10
- net +3.3V: track 0.00 -> 16.8 mm, vias 0 -> 3
- net /USB-C power controller/TPS_PP_EXT2: track 0.00 -> 16.3 mm, vias 0 -> 2
- net Net-(Q11-Pad1): track 0.00 -> 16.0 mm, vias 0 -> 1
- net Net-(J14-Pad2): track 0.00 -> 15.1 mm
- net /USB-C power controller/USB1_SOURCE_EN: track 0.00 -> 14.1 mm, vias 0 -> 1
- net /MCU_USB_D-: track 0.00 -> 13.7 mm, vias 0 -> 5
- net /USB-C power controller/USB2_SOURCE: track 0.00 -> 13.6 mm
- net Net-(J14-Pad3): track 0.00 -> 13.0 mm
- net /CP2102_USB_D-: track 0.00 -> 12.8 mm, vias 0 -> 4
- net /USB-C power controller/USB2_VBUS: track 0.06 -> 12.3 mm, vias 0 -> 25
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- added copper zone on F.Cu, net +3.3V
- added copper zone on B.Cu, net /USB-C power controller/USB1_VBUS
- added copper zone on B.Cu, net /USB-C power controller/USB2_VBUS
- added copper zone on B.Cu, net Net-(U14-Pad15)
- added copper zone on F.Cu, net Net-(U14-Pad15)
- added copper zone on B.Cu, net Net-(U14-Pad52)
- added copper zone on F.Cu, net Net-(U14-Pad52)
- added copper zone on B.Cu, net SYS VBUS

Commit message: usb power source added, need to reassemble to 4-layers
Parts:
- removed the C153 at (187.7, 77.2)
- removed the J12 at (202.2, 84.3)
- removed J13: Conn_01x03, Connector_PinSocket_2.54mm:PinSocket_1x03_P2.54mm_Vertical
- removed the J2 at (202.2, 80.7)
- added C129: 0.1uF, Capacitor_SMD:C_0603_1608Metric_Pad1.08x0.95mm_HandSolder, F.Cu at (188.9, 59.5)
- added C130: 0.1uF, Capacitor_SMD:C_0603_1608Metric_Pad1.08x0.95mm_HandSolder, F.Cu at (190.8, 153.8)
- added D17: WS2812B, LED_SMD:LED_WS2812B_PLCC4_5.0x5.0mm_P3.2mm, B.Cu at (187.4, 58.6)
- added D18: WS2812B, LED_SMD:LED_WS2812B_PLCC4_5.0x5.0mm_P3.2mm, B.Cu at (187.4, 151.3)
- added TP1: TestPoint, TestPoint:TestPoint_Pad_D1.5mm, F.Cu at (201.6, 81.6)
- added TP2: TestPoint, TestPoint:TestPoint_Pad_D1.5mm, F.Cu at (204.1, 81.6)
- added TP3: TestPoint, TestPoint:TestPoint_Pad_D1.5mm, F.Cu at (206.6, 81.6)
- added TP4: TestPoint, TestPoint:TestPoint_Pad_D1.5mm, F.Cu at (200.2, 85.7)
- added TP5: TestPoint, TestPoint:TestPoint_Pad_D1.5mm, F.Cu at (202.7, 85.7)
- added TP6: TestPoint, TestPoint:TestPoint_Pad_D1.5mm, F.Cu at (205.2, 85.7)
- added TP7: TestPoint, TestPoint:TestPoint_Pad_D1.5mm, F.Cu at (201.6, 72.0)
- added TP8: TestPoint, TestPoint:TestPoint_Pad_D1.5mm, F.Cu at (201.6, 74.5)
- added TP9: TestPoint, TestPoint:TestPoint_Pad_D1.5mm, F.Cu at (201.6, 77.0)
- C159: renamed from C156; moved to B.Cu
- C160: renamed from C157; footprint Capacitor_SMD:C_1206_3216Metric_Pad1.33x1.80mm_HandSolder -> Capacitor_SMD:C_0805_2012Metric_Pad1.18x1.45mm_HandSolder; moved to B.Cu
- C162: renamed from C159; moved to B.Cu
- C163: renamed from C160; footprint Capacitor_SMD:C_1206_3216Metric_Pad1.33x1.80mm_HandSolder -> Capacitor_SMD:C_0805_2012Metric_Pad1.18x1.45mm_HandSolder; moved to B.Cu
- C92: renamed from C91; moved to B.Cu
- C93: renamed from C92; moved to B.Cu
- C95: renamed from C94; moved to B.Cu
- C96: renamed from C95; moved to B.Cu
- C97: renamed from C96; moved to B.Cu
- D10: moved to F.Cu
- D20: renamed from D18; moved to B.Cu
- R65: moved to B.Cu
- moved C7 265.8 mm to (84.5, 106.2)
- moved C4 227.9 mm to (111.1, 132.9)
- moved C1 219.5 mm to (136.2, 135.2)
- moved C9 184.4 mm to (185.8, 135.4)
- moved RN4 176.4 mm to (198.2, 89.2)
- moved C8 163.5 mm to (211.7, 107.0)
- moved J3 158.7 mm to (191.7, 117.7)
- moved D9 141.2 mm to (62.1, 130.2), turned to 180 degrees
- moved D20 98.1 mm to (234.8, 130.2), turned to 180 degrees
- moved C147 97.3 mm to (226.4, 96.5), turned to 180 degrees
- moved D10 95.3 mm to (139.5, 104.9), turned to 90 degrees
- moved R75 90.1 mm to (229.7, 93.5), turned to 180 degrees
- moved R76 82.3 mm to (226.4, 95.0), turned to 180 degrees
- moved R68 79.3 mm to (229.7, 90.5), turned to 180 degrees
- moved C145 74.9 mm to (229.7, 92.0)
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- renumbered C99 to C100, C100 to C101, C101 to C102, C102 to C103, C103 to C104, C104 to C105, C105 to C106, C106 to C107, C107 to C108, C108 to C109, C109 to C110, C110 to C111, C111 to C112, C112 to C113, C113 to C114, C114 to C115, C115 to C116, C116 to C117, C117 to C118, C118 to C119, C119 to C120, C120 to C121, C121 to C122, C122 to C123, C123 to C124, C124 to C125, C125 to C126, C126 to C127, C127 to C128, C128 to C131, C129 to C132, C130 to C133, C131 to C134, C132 to C135, C133 to C136, C134 to C137, C135 to C138, C136 to C139, C137 to C140, C138 to C141, C139 to C142, C140 to C143, C141 to C144, C142 to C145, C143 to C146, C144 to C147, C145 to C148, C146 to C149, C147 to C150, C148 to C151, C149 to C152, C150 to C153, C151 to C154, C152 to C155, C153 to C156, C154 to C157, C155 to C158, C158 to C161, C161 to C164, C162 to C88, C88 to C89, C89 to C90, C90 to C91, C93 to C94, C97 to C98, C98 to C99, D17 to D19, J11 to J10, J14 to J11, J15 to J12, J3 to J2, J4 to J3, J5 to J4, J6 to J5, J7 to J6, J8 to J7, J9 to J8, J10 to J9
Connections:
- C131 pad 2: unconnected-(C128-Pad2) -> +5V
- D19 pad 1: unconnected-(D17-Pad1) -> +5V
- D19 pad 4: Net-(D16-Pad2) -> Net-(D19-Pad4)
- RN4 pad 6: /USB-C power controller/USB2_SOURCE_VOLTAGE_PWM -> /USB-C power controller/USB1_SOURCE_EN
- RN4 pad 7: /USB-C power controller/USB1_SOURCE_VOLTAGE_PWM -> /USB-C power controller/USB2_SOURCE_EN
- RN4 pad 8: /USB-C power controller/USB2_SOURCE_EN -> /USB-C power controller/USB1_SOURCE_VOLTAGE_PWM
- RN4 pad 9: /USB-C power controller/USB1_SOURCE_EN -> /USB-C power controller/USB2_SOURCE_VOLTAGE_PWM
Routing:
- net SYS VBUS: track 7.97 -> 105.3 mm, vias 15 -> 57
- net +5V: track 6.80 -> 82.4 mm, vias 2 -> 28
- net /USB-C power controller/USB1_SOURCE_VOLTAGE_PWM: track 0.47 -> 53.2 mm, vias 1 -> 3
- net /MCU_USB_D-: track 13.7 -> 62.3 mm, vias 5 -> 6
- net /MCU_USB_D+: track 10.2 -> 57.8 mm, vias 1 -> 2
- net /USB-C power controller/TPS_PP_EXT1: track 5.27 -> 45.5 mm, vias 1 -> 2
- net /USB-C power controller/USB1_SOURCE_EN: track 14.1 -> 50.4 mm, vias 1 -> 2
- net /BATTERY_BALANCE_EN: track 0.00 -> 32.4 mm, vias 0 -> 2
- net /BATTERY_MGMT_OTG: track 0.00 -> 28.8 mm, vias 0 -> 2
- net /USB-C power controller/USB1_CC2: track 1.86 -> 29.9 mm, vias 0 -> 6
- net /USB-C power controller/USB1_CC1: track 3.96 -> 29.8 mm, vias 0 -> 5
- net /USB-C power controller/USB2_SOURCE_EN: track 11.6 -> 35.2 mm
- net /CP2102_USB_D+: track 10.4 -> 31.1 mm, vias 0 -> 2
- net /USB-C power controller/USB2_SOURCE: track 13.6 -> 33.3 mm
- net /USB-C power controller/USB2_SOURCE_VOLTAGE_PWM: track 3.76 -> 22.9 mm
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- added copper zone on B.Cu, net +5V
- added copper zone on F.Cu, net +5V
- added copper zone on F.Cu, net /USB-C power controller/USB1_SOURCE
- added copper zone on F.Cu, net /USB-C power controller/USB2_SOURCE
- added copper zone on F.Cu, net Net-(L7-Pad1)
- added copper zone on F.Cu, net Net-(L8-Pad1)
