File: lora.kicad_sch (KiCad schematic)
At the start: 7 parts, among them U11 RA-01SH

Commit message: schematic creation
Parts:
- L5: footprint (none) -> Inductor_SMD:L_0603_1608Metric_Pad1.05x0.95mm_HandSolder
- renumbered C72 to C74, C73 to C75, C74 to C76, C75 to C77
Changed lines of the file:
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@@
   (symbol (lib_id "power:GND") (at 147.32 115.57 0) (unit 1)
     (in_bom yes) (on_board yes) (fields_autoplaced)
-    (property "Reference" "#PWR086" (id 0) (at 147.32 121.92 0)
+    (property "Reference" "#PWR092" (id 0) (at 147.32 121.92 0)
       (effects (font (size 1.27 1.27)) hide)
     )
@@
   (symbol (lib_id "Device:C") (at 143.51 83.82 90) (unit 1)
     (in_bom yes) (on_board yes)
-    (property "Reference" "C73" (id 0) (at 135.89 82.55 90))
+    (property "Reference" "C75" (id 0) (at 135.89 82.55 90))
     (property "Value" "22pF" (id 1) (at 135.89 85.09 90))
     (property "Footprint" "Capacitor_SMD:C_0603_1608Metric_Pad1.08x0.95mm_HandSolder" (id 2) (at 147.32 82.8548 0)
@@
   (symbol (lib_id "power:GND") (at 170.18 100.33 0) (unit 1)
     (in_bom yes) (on_board yes) (fields_autoplaced)
-    (property "Reference" "#PWR087" (id 0) (at 170.18 106.68 0)
+    (property "Reference" "#PWR093" (id 0) (at 170.18 106.68 0)
       (effects (font (size 1.27 1.27)) hide)
     )
@@
   (symbol (lib_id "Device:C") (at 185.42 96.52 0) (unit 1)
     (in_bom yes) (on_board yes) (fields_autoplaced)
-    (property "Reference" "C75" (id 0) (at 189.23 95.2499 0)
+    (property "Reference" "C77" (id 0) (at 189.23 95.2499 0)
       (effects (font (size 1.27 1.27)) (justify left))
     )
@@
   (symbol (lib_id "power:GND") (at 185.42 100.33 0) (unit 1)
     (in_bom yes) (on_board yes) (fields_autoplaced)
-    (property "Reference" "#PWR088" (id 0) (at 185.42 106.68 0)
+    (property "Reference" "#PWR094" (id 0) (at 185.42 106.68 0)
       (effects (font (size 1.27 1.27)) hide)
     )
@@
   (symbol (lib_id "power:GND") (at 139.7 83.82 0) (unit 1)
     (in_bom yes) (on_board yes) (fields_autoplaced)
-    (property "Reference" "#PWR084" (id 0) (at 139.7 90.17 0)
+    (property "Reference" "#PWR090" (id 0) (at 139.7 90.17 0)
       (effects (font (size 1.27 1.27)) hide)
     )
@@
   (symbol (lib_id "Device:C") (at 143.51 78.74 90) (unit 1)
     (in_bom yes) (on_board yes)
-    (property "Reference" "C72" (id 0) (at 135.89 77.47 90))
+    (property "Reference" "C74" (id 0) (at 135.89 77.47 90))
     (property "Value" "0.1uF" (id 1) (at 135.89 80.01 90))
     (property "Footprint" "Capacitor_SMD:C_0603_1608Metric_Pad1.08x0.95mm_HandSolder" (id 2) (at 147.32 77.7748 0)
@@
   (symbol (lib_id "Device:C") (at 170.18 96.52 0) (unit 1)
     (in_bom yes) (on_board yes) (fields_autoplaced)
-    (property "Reference" "C74" (id 0) (at 173.99 95.2499 0)
+    (property "Reference" "C76" (id 0) (at 173.99 95.2499 0)
       (effects (font (size 1.27 1.27)) (justify left))
     )
@@
   (symbol (lib_id "power:+3.3V") (at 147.32 78.74 0) (unit 1)
     (in_bom yes) (on_board yes) (fields_autoplaced)
-    (property "Reference" "#PWR085" (id 0) (at 147.32 82.55 0)
+    (property "Reference" "#PWR091" (id 0) (at 147.32 82.55 0)
       (effects (font (size 1.27 1.27)) hide)
     )
@@
     (property "Reference" "L5" (id 0) (at 177.8 86.36 90))
     (property "Value" "11nH" (id 1) (at 177.8 88.9 90))
-    (property "Footprint" "" (id 2) (at 177.8 92.71 0)
+    (property "Footprint" "Inductor_SMD:L_0603_1608Metric_Pad1.05x0.95mm_HandSolder" (id 2) (at 177.8 92.71 0)
       (effects (font (size 1.27 1.27)) hide)
     )
